File: peugeot_projekt.kicad_sch (KiCad schematic)
At the start: 27 parts, among them J1 ESP Power selector, J2 +12V Permanent, J3 Main Power and Data, J4 LCD Power, P1 Conn_02x20_Odd_Even, U1 ESP32, U2 LevelShifter4Shield, U3 TSS463C, U4 MCP2551-I-SN, U5 LM7805_TO220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

Commit message: Progress on v0.2 of the board
Parts:
- removed R4: 120, Resistor_SMD:R_1206_3216Metric_Pad1.30x1.75mm_HandSolder, symbol Device:R
- added J7: RUN Header 3B, Connector_PinSocket_2.54mm:PinSocket_1x02_P2.54mm_Vertical, symbol Connector:Conn_01x02_Female
- added R6: 10k, Resistor_SMD:R_0603_1608Metric_Pad0.98x0.95mm_HandSolder, symbol Device:R
- C1, C2, C3, C4, C5, C6, C7: footprint Capacitor_SMD:C_1206_3216Metric_Pad1.33x1.80mm_HandSolder -> Capacitor_SMD:C_0603_1608Metric_Pad1.08x0.95mm_HandSolder
- R1, R2, R3: footprint Resistor_SMD:R_1206_3216Metric_Pad1.30x1.75mm_HandSolder -> Resistor_SMD:R_0603_1608Metric_Pad0.98x0.95mm_HandSolder
- R5: value 10k -> 100k; footprint Resistor_SMD:R_1206_3216Metric_Pad1.30x1.75mm_HandSolder -> Resistor_SMD:R_0603_1608Metric_Pad0.98x0.95mm_HandSolder
Connections:
- net +3V3: no longer U2.3 (LV)
- net GNDD: now also J7.1 (Pin_1), R6.2; no longer R5.1
- net Wake PIN: no longer R5.2
- net at C6.1, J2.1 (Pin_1), U5.1 (VI): now also R5.1
- net RUN: now reaches U1.13 (D13)
- net RUN: now also J7.2 (Pin_2)
- net 3V3 - LVL_SHFT: now reaches U1.30 (3V3)
- net 3V3 - LVL_SHFT: now also U2.3 (LV)
- net Voltmeter: now reaches U1.6 (D32)
- net Voltmeter: now also R5.2, R6.1
Other:
- note added: "This board is designed to act as a HAT for a Raspberry Pi 3B (non plus). It would work for a 3B+, but the RUN header is not in the same place, so the power control would not work. There are 2 power rails, one for the ESP, and one for the Pi. The ESP is designed to be powered by the permanent 12 volt rail from the car, and the Pi from the VAN+ rail that comes on when the car wakes up from sleep. B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"
- note removed: "ID_SD and ID_SC PINS: These pins are reserved for HAT ID EEPROM. At boot time this I2C interface will be interrogated to look for an EEPROM that identifes the attached board and allows automagic setup of the GPIOs (and optionally, Linux drivers). DO NOT USE these pins for anything other than attaching an I2C ID EEPROM. Leave unconnected if ID EEPROM not required."
- company: (none) -> Mislav Milinković
- title: Peugeot Projekt PCB -> Peugeot Projekt PCB for 3B
- moved on the sheet: MK1, MK2, MK3, MK4
