File: ECU_comms.kicad_sch (KiCad schematic)
At the start: 10 parts, among them U1 TJA1051TK-3, U10 NTS0104GU12_115, U3 TSS463C, U8 ABM3B-8.000MHZ-B2-T

Commit message: Update bom values with actual chip names
Parts:
- C3: value 0.1uF -> 100nF; footprint Capacitor_SMD:C_0805_2012Metric_Pad1.18x1.45mm_HandSolder -> Capacitor_SMD:C_0805_2012Metric
- R9: value 4k7 -> 4.7K
Changed lines of the file:
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@@
 			)
 		)
-		(property "Value" "0.1uF"
+		(property "Value" "100nF"
 			(at 229.87 25.4 90)
 			(effects
@@
 			)
 		)
-		(property "Footprint" "Capacitor_SMD:C_0805_2012Metric_Pad1.18x1.45mm_HandSolder"
+		(property "Footprint" "Capacitor_SMD:C_0805_2012Metric"
 			(at 233.68 29.5148 0)
 			(effects
@@
 			)
 		)
-		(property "Description" "Unpolarized capacitor"
+		(property "Description" ""
 			(at 229.87 30.48 0)
 			(effects
@@
 			)
 		)
-		(property "Value" "4k7"
+		(property "Value" "4.7K"
 			(at 53.3401 59.69 0)
 			(effects
@@
 			)
 		)
-		(property "Description" "Unpolarized capacitor"
+		(property "Description" ""
 			(at 114.3 48.26 0)
 			(effects
@@
 			)
 		)
-		(property "Description" "Unpolarized capacitor"
+		(property "Description" ""
 			(at 148.59 48.26 0)
 			(effects
