File: ESP32_WROOM.kicad_sch (KiCad schematic)
At the start: 12 parts, among them J7 Programming Socket, Q1 NPN, Q2 NPN, SW1 EN, SW2 EN, U11 NTS0104GU12_115, U6 ESP32-WROOM-32E

Commit message: Update bom values with actual chip names
Parts:
- Q1, Q2: value NPN -> MMBT2222ATT3G
Changed lines of the file:
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@@
 			)
 		)
-		(property "Value" "NPN"
+		(property "Value" "MMBT2222ATT3G"
 			(at 148.59 119.3799 0)
 			(effects
@@
 			)
 		)
-		(property "Value" "NPN"
+		(property "Value" "MMBT2222ATT3G"
 			(at 148.59 99.0599 0)
 			(effects
@@
 			)
 		)
-		(property "Description" "Generic connector, single row, 01x06, script generated"
+		(property "Description" ""
 			(at 135.89 30.48 0)
 			(effects
@@
 			)
 		)
-		(property "Description" "Unpolarized capacitor"
+		(property "Description" ""
 			(at 156.21 69.85 0)
 			(effects
