File: power.kicad_sch (KiCad schematic)
At the start: 37 parts, among them U12 VTVS25ASMF-HM3-08, U13 VTVS25ASMF-HM3-08, U2 NCP691MN33T2G, U4 AP63301WU-7, U5 AP63301WU-7, U9 VTVS25ASMF-HM3-08

Commit message: Update bom values with actual chip names
Parts:
- L1, L2: value 4.7uH -> TYA40204R7M-10
Changed lines of the file:
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@@
 	(rectangle
 		(start 228.6 74.93)
-		(end 264.16 127)
+		(end 279.4 127)
 		(stroke
 			(width 0)
@@
 			)
 		)
-		(property "Description" "Unpolarized capacitor"
+		(property "Description" ""
 			(at 247.65 49.53 0)
 			(effects
@@
 			)
 		)
-		(property "Description" "Unpolarized capacitor"
+		(property "Description" ""
 			(at 128.27 40.64 0)
 			(effects
@@
 			)
 		)
-		(property "Description" "Unpolarized capacitor"
+		(property "Description" ""
 			(at 138.43 96.52 0)
 			(effects
@@
 			)
 		)
-		(property "Value" "4.7uH"
+		(property "Value" "TYA40204R7M-10"
 			(at 115.57 31.75 90)
 			(effects
@@
 			)
 		)
-		(property "Description" "Unpolarized capacitor"
+		(property "Description" ""
 			(at 160.02 96.52 0)
 			(effects
@@
 			)
 		)
-		(property "Description" "Unpolarized capacitor"
+		(property "Description" ""
 			(at 43.18 87.63 0)
 			(effects
@@
 			)
 		)
-		(property "Description" "Unpolarized capacitor"
+		(property "Description" ""
 			(at 96.52 85.09 0)
 			(effects
@@
 			)
 		)
-		(property "Description" "Unpolarized capacitor"
+		(property "Description" ""
 			(at 259.08 49.53 0)
 			(effects
@@
 			)
 		)
-		(property "Description" "Unpolarized capacitor"
+		(property "Description" ""
 			(at 43.18 31.75 0)
 			(effects
@@
 			)
 		)
-		(property "Description" "Unpolarized capacitor"
+		(property "Description" ""
 			(at 96.52 29.21 0)
 			(effects
@@
 			)
 		)
-		(property "Description" "Unpolarized capacitor"
+		(property "Description" ""
 			(at 53.34 87.63 0)
 			(effects
@@
 			)
 		)
-		(property "Description" "Unpolarized capacitor"
+		(property "Description" ""
 			(at 193.04 25.4 0)
 			(effects
@@
 			)
 		)
-		(property "Value" "4.7uH"
+		(property "Value" "TYA40204R7M-10"
 			(at 115.57 87.63 90)
 			(effects
@@
 			)
 		)
-		(property "Description" "Unpolarized capacitor"
+		(property "Description" ""
 			(at 149.86 96.52 0)
 			(effects
@@
 			)
 		)
-		(property "Description" "Unpolarized capacitor"
+		(property "Description" ""
 			(at 193.04 34.29 0)
 			(effects
@@
 			)
 		)
-		(property "Description" "Unpolarized capacitor"
+		(property "Description" ""
 			(at 138.43 40.64 0)
 			(effects
@@
 			)
 		)
-		(property "Description" "Unpolarized capacitor"
+		(property "Description" ""
 			(at 160.02 40.64 0)
 			(effects
@@
 			)
 		)
-		(property "Description" "Unpolarized capacitor"
+		(property "Description" ""
 			(at 252.73 110.49 0)
 			(effects
@@
 			)
 		)
-		(property "Description" "Unpolarized capacitor"
+		(property "Description" ""
 			(at 53.34 31.75 0)
 			(effects
@@
 			)
 		)
-		(property "Description" "Unpolarized capacitor"
+		(property "Description" ""
 			(at 128.27 96.52 0)
 			(effects
@@
 			)
 		)
-		(property "Description" "Unpolarized capacitor"
+		(property "Description" ""
 			(at 149.86 40.64 0)
 			(effects
